File: Hardware.kicad_pcb (KiCad board)
At the start: 2 copper layers, 0 parts

Commit message: added scematics for gps and sd reader
Other:
- board outline added: 30.5 x 24 mm
Changed lines of the file:
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@@
 	)
 	(net 0 "")
+	(gr_rect
+		(start 35.5 50)
+		(end 66 74)
+		(stroke
+			(width 0.05)
+			(type default)
+		)
+		(fill none)
+		(layer "Edge.Cuts")
+	)
 )
