File: Hardware.kicad_pcb (KiCad board)
At the start: 2 copper layers, 80 x 40 mm, 124 parts, among them J1 Conn_01x06_Socket, J2 JAE_SIM_Card_SF72S006, J3 Conn_Coaxial, J4 Conn_Coaxial, J5 Conn_01x05_Socket, J9 Battery, Q1 BC849, Q2 BC849, Q3 MMBT3904, Q4 BC849, Q5 MMBT3904, Q6 MMBT3904, SW1 SW_Push, SW3 SW_Push, U1 ESP32-WROOM-32, U10 MIC29302AWD, U11 AMS1117-3.3, U2 NEO-M8M, U3 SN65HVD231, U4 BQ24075RGT, U5 AT24CS01-XHM, U6 A7670E, U7 AMS1117-3.3, U8 MP1584EN

Commit message: cleaned silkscreen
Parts:
- moved H5 1.00 mm to (184.5, 66.5)
Other:
- board text added: "->"
- board text added: "<-"
Changed lines of the file:
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@@
 		(tags "resistor")
 		(property "Reference" "R51"
-			(at -2 0.5 -90)
+			(at 0 3 90)
 			(layer "F.SilkS")
 			(effects
@@
 		(tags "Diode Mini-MELF (SOD-80)")
 		(property "Reference" "D10"
-			(at 0 2 90)
+			(at 0 -2.125 90)
 			(layer "F.SilkS")
 			(effects
@@
 		(tags "capacitor")
 		(property "Reference" "C5"
-			(at 4.5 -1.5 0)
+			(at 5.5 0 0)
 			(layer "F.SilkS")
 			(effects
@@
 		(tags "resistor")
 		(property "Reference" "R4"
-			(at -2.3375 0.05 180)
+			(at -0.3375 11.05 180)
 			(layer "F.SilkS")
 			(effects
@@
 	(footprint "MountingHole:MountingHole_3.2mm_M3"
 		(layer "F.Cu")
-		(at 184.5 67.5)
+		(at 184.5 66.5)
 		(descr "Mounting Hole 3.2mm, no annular, M3")
 		(tags "mounting hole 3.2mm no annular m3")
 		(property "Reference" "H5"
-			(at 3 -4 180)
+			(at 3 -3.5 180)
 			(layer "F.SilkS")
 			(effects
@@
 		(tags "resistor")
 		(property "Reference" "R3"
-			(at 2.5 0 180)
+			(at 0.3375 -5.05 180)
 			(layer "F.SilkS")
 			(effects
@@
 		(tags "resistor")
 		(property "Reference" "R1"
-			(at 0.325 5 0)
+			(at -0.175 6 0)
 			(layer "F.SilkS")
 			(effects
@@
 		(tags "capacitor")
 		(property "Reference" "C4"
-			(at -2 -6 180)
+			(at -0.5 -6.5 180)
 			(layer "F.SilkS")
 			(effects
@@
 		(tags "capacitor")
 		(property "Reference" "C1"
-			(at 0.325 5.5 0)
+			(at -0.175 6 0)
 			(layer "F.SilkS")
 			(effects
@@
 		(tags "SOT TO_SOT_SMD")
 		(property "Reference" "Q2"
-			(at -2.4375 -0.05 180)
+			(at 0.725 8.5 180)
 			(layer "F.SilkS")
 			(effects
@@
 		(tags "Through hole pin header THT 1x06 2.54mm single row")
 		(property "Reference" "J1"
-			(at -1 15.12 -90)
+			(at 2 13.12 0)
 			(layer "F.SilkS")
 			(effects
@@
 		(tags "resistor")
 		(property "Reference" "R52"
-			(at 3 0 90)
+			(at 3 1 90)
 			(layer "F.SilkS")
 			(effects
@@
 		(tags "SOT TO_SOT_SMD")
 		(property "Reference" "Q1"
-			(at -2.4375 -0.05 0)
+			(at 0.725 7.5 0)
 			(layer "F.SilkS")
 			(effects
@@
 		(tags "capacitor")
 		(property "Reference" "C38"
-			(at 0 2 180)
+			(at -9.6 1 180)
 			(layer "B.SilkS")
 			(effects
@@
 		(tags "capacitor")
 		(property "Reference" "C19"
-			(at -0.6875 3.05 90)
+			(at -0.1875 3.55 90)
 			(layer "B.SilkS")
 			(effects
@@
 		(tags "capacitor")
 		(property "Reference" "C11"
-			(at 5 -0.3625 180)
+			(at 5 -1 180)
 			(layer "B.SilkS")
 			(effects
@@
 		(tags "capacitor")
 		(property "Reference" "D7"
-			(at 2.775 0 90)
+			(at 2.275 0 90)
 			(layer "B.SilkS")
 			(effects
@@
 		(tags "capacitor")
 		(property "Reference" "C30"
-			(at 0 -3 90)
+			(at 0 -1.6625 90)
 			(layer "B.SilkS")
 			(effects
@@
 		(tags "capacitor")
 		(property "Reference" "C37"
-			(at 0 -2 0)
+			(at 8.6 -1 0)
 			(layer "B.SilkS")
 			(effects
@@
 		(tags "VQFN NoLead")
 		(property "Reference" "U4"
-			(at 3.0625 1.4375 -90)
+			(at 3.0625 -0.1 -90)
 			(layer "B.SilkS")
 			(effects
@@
 		(tags "capacitor")
 		(property "Reference" "C36"
-			(at 0 -1.5 180)
+			(at -9.6 9 180)
 			(layer "B.SilkS")
 			(effects
@@
 		(tags "resistor")
 		(property "Reference" "R13"
-			(at 1.8625 4 90)
+			(at 2 6 180)
 			(layer "B.SilkS")
 			(effects
@@
 		(tags "capacitor")
 		(property "Reference" "C35"
-			(at 0 1.85 0)
+			(at 8.6 -9.15 0)
 			(layer "B.SilkS")
 			(effects
@@
 		(tags "resistor")
 		(property "Reference" "R2"
-			(at 2.775 0 90)
+			(at 2.275 0 90)
 			(layer "B.SilkS")
 			(effects
@@
 		(tags "capacitor")
 		(property "Reference" "C16"
-			(at -3.5 0 -90)
+			(at -3 0 -90)
 			(layer "B.SilkS")
 			(effects
@@
 		(tags "SOT TO_SOT_SMD")
 		(property "Reference" "D3"
-			(at 0 2.5 0)
+			(at 3 1.5 90)
 			(layer "B.SilkS")
 			(effects
@@
 		(tags "resistor")
 		(property "Reference" "R10"
-			(at -0.6375 3.55 90)
+			(at -0.1375 4.05 90)
 			(layer "B.SilkS")
 			(effects
@@
 		(tags "capacitor")
 		(property "Reference" "C39"
-			(at 4.125 0.125 90)
+			(at 0 -1.6625 90)
 			(layer "B.SilkS")
 			(effects
@@
 		(tags "resistor")
 		(property "Reference" "R5"
-			(at 2.775 0 90)
+			(at 2.275 0 90)
 			(layer "B.SilkS")
 			(effects
@@
 		(tags "capacitor")
 		(property "Reference" "D8"
-			(at 2.775 0 90)
+			(at 2.275 0 90)
 			(layer "B.SilkS")
 			(effects
@@
 		(tags "capacitor")
 		(property "Reference" "C10"
-			(at 3.5 -2 0)
+			(at 3.5 -1.1375 0)
 			(layer "B.SilkS")
 			(effects
@@
 		(layer "Edge.Cuts")
 	)
+	(gr_text "<-"
+		(at 133 88.5 180)
+		(layer "B.SilkS")
+		(effects
+			(font
+				(size 1 1)
+				(thickness 0.1)
+			)
+			(justify left bottom mirror)
+		)
+	)
+	(gr_text "->"
+		(at 178 65 -90)
+		(layer "F.SilkS")
+		(effects
+			(font
+				(size 1 1)
+				(thickness 0.1)
+			)
+			(justify left bottom)
+		)
+	)
+	(gr_text "<-"
+		(at 176 97.5 0)
+		(layer "F.SilkS")
+		(effects
+			(font
+				(size 1 1)
+				(thickness 0.1)
+			)
+			(justify left bottom)
+		)
+	)
 	(via
