File: SD_Modula.kicad_sch (KiCad schematic)
At the start: 7 parts, among them J6 Micro_SD_Card, U8 AMS1117-3.3

Commit message: pre remobing sd card
Parts:
- TP18: footprint TestPoint:TestPoint_Pad_D2.0mm -> TestPoint:TestPoint_Pad_D1.5mm
Changed lines of the file:
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@@
 			)
 		)
-		(property "Footprint" "TestPoint:TestPoint_Pad_D2.0mm"
+		(property "Footprint" "TestPoint:TestPoint_Pad_D1.5mm"
 			(at 179.07 30.48 0)
 			(effects
